File: Modules/Sensor/TemperatureReader/EagleDesigns/TemperatureReader.sch (EAGLE design)
At the start: 6 parts, among them U1 TINY85-20-DIP, U2 MLX90614_

Commit message: added eagle files for #31
Parts:
- added C2: 22pF, adafruit:C-USC0603
- added C3: 0.22uF, adafruit:C-USC0402
- added JP2: (no value), SparkFun-Connectors:M03PTH
- added R4: 4.7K, adafruit:R-US_R0603
- added U$2: NX503, MakerWear:NX503
- C1: value 0.22uF -> 22pF; device adafruit:C-USC0402 -> adafruit:C-USC0603
- R2: value 4.7K -> 10K; device adafruit:R-US_R0603 -> resistor:R-US_R0603
- U1: value TINY85-20-DIP -> MLX90614; device SparkFun-DigitalIC:ATTINY45TINY85-20-DIP -> MakerWear:MLX90614
- U2: value MLX90614_ -> ATMEGA328P_TQFP; device SparkFun-Sensors:MLX90614_ -> SparkFun-DigitalIC:ATMEGA328P_TQFP
Connections:
- removed net NRES: U1.PB5(NRES)
- removed net OUT(MISO): R2.2, U1.PB1(MISO)
- removed net SCK: U1.PB2(SCK/ADC1), U2.SCL/VZ
- removed net SDA(MOSI): U1.PB0(MOSI), U2.PWM/SDA
- new net 1X3SIN-SOUT: JP1.1, JP1.4, R1.2
- new net N$1: C1.1, U$2.P$1, U2.PB6(XTAL1/TOSC1)
- new net N$3: C2.1, U$2.P$2, U2.PB7(XTAL2/TOSC2)
- new net OUT: R4.2, U2.PB1(OC1A)
- new net RESET: JP2.1, R2.1, U2.PC6(/RESET)
- new net RX: JP2.2, U2.PD0(RXD)
- new net SCL: U1.SCL/VZ, U2.PC5(ADC5/SCL)
- new net SDA: U1.PWM/SDA, U2.PC4(ADC4/SDA)
- new net TX: JP2.3, U2.PD1(TXD)
- net 1X3SIN: now also U2.PC0(ADC0); no longer JP1.4, R1.2, U1.PB3(ADC3)
- net 1X3SOUT: now also C3.1, R4.1; no longer C1.2, JP1.1, R2.1
- net GND: now also C1.2, C2.2, C3.2, U1.VSS, U2.AGND, U2.GND@3, U2.GND@5; no longer C1.1, U1.GND, U2.VSS
- net VCC: now also R2.2, U1.VDD, U2.AVCC, U2.VCC@4, U2.VCC@6; no longer U1.VCC, U2.VDD
Other:
- moved on the sheet: C1, JP1, R1, R2

Commit message: Revert "Merge branch 'version-1.2'"
This reverts commit 982d9c85d5bd00c48b539e840003de48d3cf178d, reversing
changes made to b3895ae538c161df72313035d3e956c7a5ec4dbc.
Parts:
- removed C2: 22pF, adafruit:C-USC0603
- removed C3: 0.22uF, adafruit:C-USC0402
- removed JP2: (no value), SparkFun-Connectors:M03PTH
- removed R4: 4.7K, adafruit:R-US_R0603
- removed U$2: NX503, MakerWear:NX503
- C1: value 22pF -> 0.22uF; device adafruit:C-USC0603 -> adafruit:C-USC0402
- R2: value 10K -> 4.7K; device resistor:R-US_R0603 -> adafruit:R-US_R0603
- U1: value MLX90614 -> TINY85-20-DIP; device MakerWear:MLX90614 -> SparkFun-DigitalIC:ATTINY45TINY85-20-DIP
- U2: value ATMEGA328P_TQFP -> MLX90614_; device SparkFun-DigitalIC:ATMEGA328P_TQFP -> SparkFun-Sensors:MLX90614_
Connections:
- removed net 1X3SIN-SOUT: JP1.1, JP1.4, R1.2
- removed net N$1: C1.1, U$2.P$1, U2.PB6(XTAL1/TOSC1)
- removed net N$3: C2.1, U$2.P$2, U2.PB7(XTAL2/TOSC2)
- removed net OUT: R4.2, U2.PB1(OC1A)
- removed net RESET: JP2.1, R2.1, U2.PC6(/RESET)
- removed net RX: JP2.2, U2.PD0(RXD)
- removed net SCL: U1.SCL/VZ, U2.PC5(ADC5/SCL)
- removed net SDA: U1.PWM/SDA, U2.PC4(ADC4/SDA)
- removed net TX: JP2.3, U2.PD1(TXD)
- new net NRES: U1.PB5(NRES)
- new net OUT(MISO): R2.2, U1.PB1(MISO)
- new net SCK: U1.PB2(SCK/ADC1), U2.SCL/VZ
- new net SDA(MOSI): U1.PB0(MOSI), U2.PWM/SDA
- net 1X3SIN: now also JP1.4, R1.2, U1.PB3(ADC3); no longer U2.PC0(ADC0)
- net 1X3SOUT: now also C1.2, JP1.1, R2.1; no longer C3.1, R4.1
- net GND: now also C1.1, U1.GND, U2.VSS; no longer C1.2, C2.2, C3.2, U1.VSS, U2.AGND, U2.GND@3, U2.GND@5
- net VCC: now also U1.VCC, U2.VDD; no longer R2.2, U1.VDD, U2.AVCC, U2.VCC@4, U2.VCC@6
Other:
- moved on the sheet: C1, JP1, R1, R2
