File: Modules/Modifier/Inverter/EagleDesigns/Inverter.sch (EAGLE design)
At the start: 6 parts, among them U1 TINY85-20-DIP

Commit message: changed 0403 cap to 0603 SMD cap
to solder without difficulty!
Parts:
- C1: device adafruit:C-USC0402 -> adafruit:C-USC0603
Connections:
- net 1X3SOUT: now also C1.1; no longer C1.2
- net GND: now also C1.2; no longer C1.1
Other:
- moved on the sheet: C1
Changed lines of the file:
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@@
 <part name="R1" library="adafruit" deviceset="R-US_" device="R0603" value="1M"/>
 <part name="R2" library="adafruit" deviceset="R-US_" device="R0603" value="4.7K"/>
-<part name="C1" library="adafruit" deviceset="C-US" device="C0402" value="0.22uF"/>
+<part name="C1" library="adafruit" deviceset="C-US" device="C0603" value="0.22uF"/>
 </parts>
 <sheets>
@@
 <instance part="R1" gate="G$1" x="53.34" y="-5.08" rot="R90"/>
 <instance part="R2" gate="G$1" x="177.8" y="7.62" rot="R180"/>
-<instance part="C1" gate="G$1" x="190.5" y="-5.08" rot="R180"/>
+<instance part="C1" gate="G$1" x="190.5" y="-2.54"/>
 </instances>
 <busses>
@@
 <wire x1="190.5" y1="-7.62" x2="190.5" y2="-15.24" width="0.1524" layer="91"/>
 <pinref part="GND3" gate="1" pin="GND"/>
-<pinref part="C1" gate="G$1" pin="1"/>
+<pinref part="C1" gate="G$1" pin="2"/>
 </segment>
 <segment>
@@
 <junction x="190.5" y="7.62"/>
 <pinref part="R2" gate="G$1" pin="1"/>
-<pinref part="C1" gate="G$1" pin="2"/>
+<pinref part="C1" gate="G$1" pin="1"/>
 </segment>
 </net>
