File: Modules/Sensor/TemperatureSensor/EagleDesigns/TemperatureSensor.sch (EAGLE design)
At the start: 7 parts, among them U1 TINY85-20-DIP

Commit message: re-organized files after Merge
Parts:
- removed C1: 0.22uF, adafruit:C-USC0402
- removed R2: 4.7K, adafruit:R-US_R0603
- added C3: 0.22uF, adafruit:C-USC0603
- added R4: 4.7K, adafruit:R-US_R0603
- U1: value TINY85-20-DIP -> MLX90614; device SparkFun-DigitalIC:ATTINY45TINY85-20-DIP -> MakerWear:MLX90614
- U2: value (none) -> ATMEGA328P_TQFP; device SparkFun-Sensors:TMP36GT9 -> SparkFun-DigitalIC:ATMEGA328P_TQFP
Connections:
- removed net NRES: JP2.1, U1.PB5(NRES)
- removed net OUT(MISO): JP2.3, R2.2, U1.PB1(MISO)
- removed net SENSOR: U1.PB4(ADC2), U2.VOUT
- new net MISO: JP2.3, U2.PB4(MISO)
- new net OUT: R4.2, U2.PB1(OC1A)
- new net RESET: JP2.1, U2.PC6(/RESET)
- new net SCL: U1.SCL/VZ, U2.PC5(ADC5/SCL)
- new net SDA: U1.PWM/SDA, U2.PC4(ADC4/SDA)
- net 1X3SIN: now also U2.PC0(ADC0); no longer U1.PB3(ADC3)
- net 1X3SOUT: now also C3.1, R4.1; no longer C1.2, R2.1
- net GND: now also C3.2, U1.VSS, U2.AGND, U2.GND@3, U2.GND@5; no longer C1.1, U1.GND, U2.GND
- net MOSI: now also U2.PB3(MOSI/OC2); no longer U1.PB0(MOSI)
- net SCK: now also U2.PB5(SCK); no longer U1.PB2(SCK/ADC1)
- net VCC: now also U1.VDD, U2.AVCC, U2.VCC@4, U2.VCC@6; no longer U1.VCC, U2.VCC
Other:
- moved on the sheet: JP2, R1
