File: Modules/Misc/ProgrammableOLED_v2/EagleDesigns/ProgrammableOLED.sch (EAGLE design)
At the start: 17 parts, among them U2 ATMEGA328P_TQFP

Commit message: updated the top PCB of the programmable module with a bigger PCB
TODO: iterate and refine the top PCB
Parts:
- removed JP2: (no value), SparkFun-Connectors:M04PTH
- JP1: device SparkFun-Connectors:M04PTH -> SparkFun-Connectors:M04X2
Connections:
- net GND: now also JP1.8; no longer JP2.1
- net SIN1: now also JP1.6; no longer JP2.2
- net SIN2: now also JP1.4; no longer JP2.3
- net SIN3: now also JP1.2; no longer JP2.4
- net SOUT2: now also JP1.5; no longer JP1.2
- net SOUT3: now also JP1.7; no longer JP1.1
- net VCC: now also JP1.1; no longer JP1.4
Other:
- moved on the sheet: C1, C2, C3, C4, C5, OLED1, R1, R2, R3, R4, R5, R6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
