File: Modules/Misc/Programmable/EagleDesigns/Programmable.sch (EAGLE design)
At the start: 12 parts, among them U2 ATMEGA328P_TQFP

Commit message: Added programmable module's top PCB
Parts:
- added JP3: (no value), SparkFun-Connectors:M04PTH
Connections:
- net GND: now also JP2.1
- net MISO: now also JP3.2
- net MOSI: now also JP3.1
- net OUT1: now also U2.PD5(T1); no longer U2.PB1(OC1A)
- net OUT2: now also U2.PB1(OC1A); no longer U2.PB2(SS/OC1B)
- net OUT3: now also U2.PB2(SS/OC1B); no longer U2.PD5(T1)
- net RESET: now also JP3.4
- net SCK: now also JP3.3
- net SIN1: now also JP2.2
- net SIN2: now also JP2.3
- net SIN3: now also JP2.4
- net SOUT1: now also JP1.3
- net SOUT2: now also JP1.2
- net SOUT3: now also JP1.1
- net VCC: now also JP1.4
Other:
- moved on the sheet: C1, C2, C3, JP2, R1, R2, R3, R4, R5, R6, U2

Commit message: added the programmable module (without OLED display)
Parts:
- removed JP2, JP3: (no value), SparkFun-Connectors:M04PTH
- added JP5: (no value), SparkFun-Connectors:USB-ABCONN-11794
- JP1: device SparkFun-Connectors:M04PTH -> SparkFun-Connectors:M04X2
Connections:
- removed net MISO: JP3.2, U2.PB4(MISO)
- removed net MOSI: JP3.1, U2.PB3(MOSI/OC2)
- removed net SCK: JP3.3, U2.PB5(SCK)
- new net RX: JP5.USBID, U2.PD0(RXD)
- new net TX: JP5.D+, U2.PD1(TXD)
- net GND: now also JP1.8, JP5.GND, JP5.SHIELD; no longer JP2.1
- net OUT1: now also U2.PD3(INT1); no longer U2.PD5(T1)
- net OUT2: now also U2.PD5(T1); no longer U2.PB1(OC1A)
- net OUT3: now also U2.PD6(AIN0); no longer U2.PB2(SS/OC1B)
- net RESET: now also JP5.D-; no longer JP3.4
- net SIN1: now also JP1.6; no longer JP2.2
- net SIN2: now also JP1.4; no longer JP2.3
- net SIN3: now also JP1.2; no longer JP2.4
- net SOUT2: now also JP1.5; no longer JP1.2
- net SOUT3: now also JP1.7; no longer JP1.1
- net VCC: now also JP1.1, JP5.VBUS; no longer JP1.4
Other:
- moved on the sheet: C1, C2, C3, R1, R2, R3, R4, R5, R6, U2
