File: Modules/Misc/Programmable/EagleDesigns/Programmable.brd (EAGLE design)
At the start: 100 x 80 mm, 12 parts, among them U2 ATMEGA328P_TQFP

Commit message: another round of minor fixes
Routing:
- net VCC: track 35.9 -> 36.6 mm
- net RESET: track 8.67 -> 8.04 mm
Changed lines of the file:
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@@
 <layer number="21" name="tPlace" color="7" fill="1" visible="no" active="yes"/>
 <layer number="22" name="bPlace" color="7" fill="1" visible="no" active="yes"/>
-<layer number="23" name="tOrigins" color="15" fill="1" visible="yes" active="yes"/>
-<layer number="24" name="bOrigins" color="15" fill="1" visible="yes" active="yes"/>
+<layer number="23" name="tOrigins" color="15" fill="1" visible="no" active="yes"/>
+<layer number="24" name="bOrigins" color="15" fill="1" visible="no" active="yes"/>
 <layer number="25" name="tNames" color="7" fill="1" visible="no" active="yes"/>
 <layer number="26" name="bNames" color="7" fill="1" visible="no" active="yes"/>
@@
 <layer number="112" name="tSilk" color="7" fill="1" visible="no" active="yes"/>
 <layer number="113" name="IDFDebug" color="4" fill="1" visible="no" active="yes"/>
-<layer number="114" name="Badge_Outline" color="7" fill="1" visible="yes" active="yes"/>
-<layer number="115" name="ReferenceISLANDS" color="7" fill="1" visible="yes" active="yes"/>
+<layer number="114" name="Badge_Outline" color="7" fill="1" visible="no" active="yes"/>
+<layer number="115" name="ReferenceISLANDS" color="7" fill="1" visible="no" active="yes"/>
 <layer number="116" name="Patch_BOT" color="9" fill="4" visible="no" active="yes"/>
-<layer number="118" name="Rect_Pads" color="7" fill="1" visible="yes" active="yes"/>
+<layer number="118" name="Rect_Pads" color="7" fill="1" visible="no" active="yes"/>
 <layer number="121" name="_tsilk" color="7" fill="1" visible="no" active="yes"/>
 <layer number="122" name="_bsilk" color="7" fill="1" visible="no" active="yes"/>
@@
 <layer number="127" name="_tValues" color="7" fill="1" visible="no" active="yes"/>
 <layer number="128" name="_bValues" color="7" fill="1" visible="no" active="yes"/>
-<layer number="129" name="Mask" color="7" fill="1" visible="yes" active="yes"/>
+<layer number="129" name="Mask" color="7" fill="1" visible="no" active="yes"/>
 <layer number="131" name="tAdjust" color="7" fill="1" visible="no" active="yes"/>
 <layer number="132" name="bAdjust" color="7" fill="1" visible="no" active="yes"/>
@@
 <layer number="223" name="223bmp" color="24" fill="1" visible="no" active="no"/>
 <layer number="224" name="224bmp" color="25" fill="1" visible="no" active="no"/>
-<layer number="225" name="225bmp" color="7" fill="1" visible="yes" active="yes"/>
-<layer number="226" name="226bmp" color="7" fill="1" visible="yes" active="yes"/>
-<layer number="227" name="227bmp" color="7" fill="1" visible="yes" active="yes"/>
-<layer number="228" name="228bmp" color="7" fill="1" visible="yes" active="yes"/>
-<layer number="229" name="229bmp" color="7" fill="1" visible="yes" active="yes"/>
-<layer number="230" name="230bmp" color="7" fill="1" visible="yes" active="yes"/>
-<layer number="231" name="231bmp" color="7" fill="1" visible="yes" active="yes"/>
+<layer number="225" name="225bmp" color="7" fill="1" visible="no" active="yes"/>
+<layer number="226" name="226bmp" color="7" fill="1" visible="no" active="yes"/>
+<layer number="227" name="227bmp" color="7" fill="1" visible="no" active="yes"/>
+<layer number="228" name="228bmp" color="7" fill="1" visible="no" active="yes"/>
+<layer number="229" name="229bmp" color="7" fill="1" visible="no" active="yes"/>
+<layer number="230" name="230bmp" color="7" fill="1" visible="no" active="yes"/>
+<layer number="231" name="231bmp" color="7" fill="1" visible="no" active="yes"/>
 <layer number="232" name="Eagle3D_PG2" color="7" fill="1" visible="no" active="no"/>
 <layer number="233" name="Eagle3D_PG3" color="7" fill="1" visible="no" active="no"/>
@@
 <layer number="251" name="SMDround" color="12" fill="11" visible="no" active="no"/>
 <layer number="254" name="cooling" color="7" fill="1" visible="no" active="yes"/>
-<layer number="255" name="routoute" color="7" fill="1" visible="yes" active="yes"/>
+<layer number="255" name="routoute" color="7" fill="1" visible="no" active="yes"/>
 </layers>
 <board>
@@
 <wire x1="15.6" y1="22.3526" x2="15.69" y2="22.2626" width="0.254" layer="16"/>
 <wire x1="10.57" y1="4.1" x2="8.61" y2="6.06" width="0.254" layer="16"/>
-<wire x1="8.61" y1="6.06" x2="8.62" y2="11.64" width="0.254" layer="16"/>
-<wire x1="8.62" y1="11.64" x2="8.23" y2="12.08" width="0.254" layer="16"/>
-<via x="8.23" y="12.08" extent="1-16" drill="0.3" diameter="0.254"/>
+<via x="8.19" y="13.09" extent="1-16" drill="0.3" diameter="0.254"/>
 <wire x1="14.09" y1="15.95" x2="15.2" y2="15.95" width="0.254" layer="1"/>
-<wire x1="8.91" y1="12.76" x2="9.24" y2="13.09" width="0.254" layer="1"/>
 <wire x1="14.09" y1="15.95" x2="11.125" y2="13.195" width="0.254" layer="1"/>
 <wire x1="15.2" y1="15.95" x2="15.7" y2="16.45" width="0.254" layer="1"/>
@@
 <wire x1="16.96" y1="19.79" x2="15.71" y2="19.79" width="0.254" layer="1"/>
 <wire x1="15.71" y1="16.64" x2="15.71" y2="19.79" width="0.254" layer="16"/>
-<wire x1="9.24" y1="13.09" x2="11.02" y2="13.09" width="0.254" layer="1"/>
+<wire x1="8.19" y1="13.09" x2="11.02" y2="13.09" width="0.254" layer="1"/>
 <wire x1="11.02" y1="13.09" x2="11.125" y2="13.195" width="0.254" layer="1"/>
-<wire x1="8.91" y1="12.76" x2="8.62" y2="12.46" width="0.254" layer="1"/>
-<wire x1="8.62" y1="12.46" x2="8.23" y2="12.08" width="0.254" layer="1"/>
+<wire x1="8.19" y1="13.09" x2="8.19" y2="9.9" width="0.254" layer="16"/>
+<wire x1="8.19" y1="9.9" x2="8.61" y2="9.48" width="0.254" layer="16"/>
+<wire x1="8.61" y1="9.48" x2="8.61" y2="6.06" width="0.254" layer="16"/>
 </signal>
 <signal name="RESET">
@@
 <wire x1="10.1074" y1="18.46" x2="11.04" y2="18.46" width="0.254" layer="16"/>
 <via x="12.95" y="16.98" extent="1-16" drill="0.3" diameter="0.254"/>
-<wire x1="14.76" y1="16.54" x2="15.06" y2="16.84" width="0.254" layer="1"/>
-<wire x1="15.06" y1="16.84" x2="15.06" y2="19.64" width="0.254" layer="1"/>
-<wire x1="14.76" y1="16.54" x2="13.39" y2="16.54" width="0.254" layer="1"/>
-<wire x1="13.39" y1="16.54" x2="12.95" y2="16.98" width="0.254" layer="1"/>
-<wire x1="11.04" y1="18.46" x2="12.27" y2="17.23" width="0.254" layer="16"/>
-<wire x1="12.27" y1="17.23" x2="12.7" y2="17.23" width="0.254" layer="16"/>
-<wire x1="12.7" y1="17.23" x2="12.95" y2="16.98" width="0.254" layer="16"/>
+<wire x1="14.74" y1="16.98" x2="12.95" y2="16.98" width="0.254" layer="1"/>
+<wire x1="11.04" y1="18.46" x2="12.52" y2="16.98" width="0.254" layer="16"/>
+<wire x1="12.52" y1="16.98" x2="12.95" y2="16.98" width="0.254" layer="16"/>
+<wire x1="14.74" y1="16.98" x2="15.06" y2="17.3" width="0.254" layer="1"/>
+<wire x1="15.06" y1="17.3" x2="15.06" y2="19.64" width="0.254" layer="1"/>
 </signal>
 <signal name="OUT1">
@@
 <via x="11.92" y="20.69" extent="1-16" drill="0.3" diameter="0.254"/>
 <wire x1="10.1174" y1="20.05" x2="10.1374" y2="20.03" width="0.254" layer="16"/>
-<wire x1="11.92" y1="20.69" x2="14.4" y2="20.69" width="0.254" layer="1"/>
-<wire x1="14.4" y1="20.69" x2="14.41" y2="19.64" width="0.254" layer="1"/>
+<wire x1="14.4" y1="20.93" x2="14.41" y2="19.64" width="0.254" layer="1"/>
 <wire x1="11.92" y1="20.69" x2="11.92" y2="20.06" width="0.254" layer="16"/>
 <wire x1="11.92" y1="20.06" x2="11.59" y2="20.06" width="0.254" layer="16"/>
 <wire x1="11.59" y1="20.06" x2="10.1174" y2="20.05" width="0.254" layer="16"/>
 <wire x1="10.1174" y1="20.05" x2="10.1074" y2="20.06" width="0.254" layer="16"/>
+<wire x1="14.4" y1="20.93" x2="12.16" y2="20.93" width="0.254" layer="1"/>
+<wire x1="12.16" y1="20.93" x2="11.92" y2="20.69" width="0.254" layer="1"/>
 </signal>
 </signals>
