File: Modules/Misc/ProgrammableOLED/EagleDesigns/ProgrammableOLED.sch (EAGLE design)
At the start: 14 parts, among them U2 ATMEGA328P_TQFP

Commit message: deleted the other incomplete programmable module
Parts:
- removed JP2: (no value), SparkFun-Connectors:M04PTH
- removed JP4: (no value), SparkFun-Connectors:USB_MICROB_PLUGCONN-11752
- removed U$1: OLED, MakerWear:OLED
- added C4, C5: 1uF X5R, SparkFun-Passives:CAP0805
- added JP5: (no value), SparkFun-Connectors:USB-ABCONN-11794
- added OLED1: OLED0.66, microView-temp:OLED0.66
- added R7: 390k, SparkFun-Passives:RESISTOR0603-RES
- JP1: device SparkFun-Connectors:M04PTH -> SparkFun-Connectors:M04X2
Connections:
- removed net OLED_CLK: U$1.CLOCK
- removed net OLED_CS: U$1.CS
- removed net OLED_DATA: U$1.DATA_IN
- removed net OLED_RESET: U$1.RESET
- removed net OLED_RS: U$1.RS
- new net C1N: C4.2, OLED1.C1N
- new net C1P: C4.1, OLED1.C1P
- new net C2N: C5.2, OLED1.C2N
- new net C2P: C5.1, OLED1.C2P
- new net IREF: OLED1.IREF, R7.2
- new net OLED-CS: OLED1.!CS!, U2.PB2(SS/OC1B)
- new net OLED-D/C: OLED1.D/!C!, U2.PB0(ICP)
- new net OLED-MOSI: OLED1.D1/MOSI, U2.PB3(MOSI/OC2)
- new net OLED-RST: OLED1.!RESET!, U2.PB1(OC1A)
- new net OLED-SCK: OLED1.D0/SCK, U2.PB5(SCK)
- net GND: now also JP1.8, JP5.GND, JP5.SHIELD, OLED1.BS1, OLED1.BS2, OLED1.GND@1, OLED1.GND@2, OLED1.VLSS, OLED1.VSS, R7.1; no longer JP2.1, JP4.GND, JP4.SHIELD, U$1.GND1, U$1.GND2
- net OUT1: now also U2.PD3(INT1); no longer U2.PD5(T1)
- net OUT2: now also U2.PD5(T1); no longer U2.PB1(OC1A)
- net OUT3: now also U2.PD6(AIN0); no longer U2.PB2(SS/OC1B)
- net RESET: now also JP5.D-; no longer JP4.ID
- net RX: now also JP5.USBID; no longer JP4.D-
- net SIN1: now also JP1.6; no longer JP2.2
- net SIN2: now also JP1.4; no longer JP2.3
- net SIN3: now also JP1.2; no longer JP2.4
- net SOUT2: now also JP1.5; no longer JP1.2
- net SOUT3: now also JP1.7; no longer JP1.1
- net TX: now also JP5.D+; no longer JP4.D+
- net VCC: now also JP1.1, JP5.VBUS, OLED1.VBAT, OLED1.VDD; no longer JP1.4, JP4.VCC, U$1.3.3V
Other:
- moved on the sheet: C1, C2, C3, R1, R2, R3, R4, R5, R6, U2
